Commit message: 新模型

File: src/manipulator/urdf/manipulator.urdf (robot description, URDF)
Before this commit: robot manipulator, 10 links, 9 joints
Links:
- removed link tool
- link base_link: mass 0.0001 -> 0.51184
- link link1: mass 0.0001 -> 0.11922
- link link2: mass 0.0001 -> 0.13979
- link link3: mass 0.0001 -> 0.084191
- link link4: mass 0.0001 -> 0.12668
- link link5: mass 0.0001 -> 0.085932
- link link6: mass 0.0001 -> 0.091478
- link link7: mass 0.0001 -> 0.19202
Joints:
- removed joint tool_
- joint joint1: axis 0 1 0 -> 0 0 1; limit lower=-3.14 upper=3.14 effort=100 velocity=1 -> lower=-3.14 upper=3.14 effort=1000 velocity=1000; origin xyz=0 0 0 rpy=-1.5708 0 -0.8318 -> xyz=0 0 0.068 rpy=0 0 0; type continuous -> revolute
- joint joint2: axis 0 1 0 -> 0 0 1; limit lower=-3.14 upper=3.14 effort=100 velocity=1 -> lower=-1.55 upper=1.55 effort=1000 velocity=1000; origin xyz=0 -0.0800000000000001 0 rpy=2.19762652073232 0.421087201612375 1.05699155584512 -> xyz=0.0005 0 0 rpy=0 -1.5708 0; type continuous -> revolute
- joint joint3: axis 0 1 0 -> 0 0 1; limit lower=-3.14 upper=3.14 effort=100 velocity=1 -> lower=-3.14 upper=3.14 effort=1000 velocity=1000; origin xyz=-0.019243 -0.0005 0.014693 rpy=-2.33 -0.57973 1.0473 -> xyz=0.206 0 0 rpy=0 1.5708 0; type continuous -> revolute
- joint joint4: axis 0 1 0 -> 0 0 1; limit lower=-3.14 upper=3.14 effort=100 velocity=1 -> lower=-1.55 upper=1.55 effort=1000 velocity=1000; origin xyz=0 -0.18179 0 rpy=2.3788 0.070271 1.5038 -> xyz=-0.003 0 0 rpy=0 -1.5708 0; type continuous -> revolute
- joint joint5: axis 0 1 0 -> 0 0 1; limit lower=-3.14 upper=3.14 effort=100 velocity=1 -> lower=-3.14 upper=3.14 effort=1000 velocity=1000; origin xyz=-0.032343 0.003 0.0031491 rpy=-0.10266 -0.33137 -1.5373 -> xyz=0.182 0 0 rpy=0 1.5708 0; type continuous -> revolute
- joint joint6: axis 0 1 0 -> 0 0 1; limit lower=-3.14 upper=3.14 effort=100 velocity=1 -> lower=-1.55 upper=1.55 effort=1000 velocity=1000; origin xyz=0 -0.1495 0 rpy=0.47997 0.78426 1.9231 -> xyz=0 0 0 rpy=0 -1.5708 0; type continuous -> revolute
- joint joint7: axis 1 0 0 -> 0 0 1; limit lower=-3.14 upper=3.14 effort=100 velocity=1 -> lower=-3.14 upper=3.14 effort=1000 velocity=1000; origin xyz=-0.035277 0 -0.039681 rpy=-0.20886 0.84408 3.1416 -> xyz=0.1161 0 0 rpy=0 1.5708 0; type continuous -> revolute

Commit message: 123

File: src/manipulator/urdf/manipulator.urdf (robot description, URDF)
Before this commit: robot manipulator, 9 links, 8 joints
Joints:
- joint joint4: limit lower=-1.55 upper=1.55 effort=1000 velocity=1000 -> lower=-1.3 upper=1.3 effort=1000 velocity=1000
